File: hardware/KiCad/schematics/mimeofreq.kicad_sch (KiCad schematic)
At the start: 19 parts, among them J1 AudioJack2, J2 AudioJack2, J3 Jack-DC, SW1 SW_SPST, SW2 SW_SPST, SW3 SW_SPDT

Commit message: Added identification properties for KiCad schematic drawing sheets.
Connections:
- net POT1: now also A1.26 (ADC_4); no longer A1.22 (ADC_0)
- net POT2: now also A1.25 (ADC_3); no longer A1.23 (ADC_1)
- net POT4: now also A1.23 (ADC_1); no longer A1.25 (ADC_3)
- net POT5: now also A1.22 (ADC_0); no longer A1.26 (ADC_4)
Other:
- company: (none) -> github.com/patrick-electrick
- title: (none) -> MIMEOFREQ
Changed lines of the file:
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@@
 	(generator_version "10.0")
 	(paper "A4")
+	(title_block
+		(title "MIMEOFREQ")
+		(date "2026-10-21")
+		(rev "1")
+		(company "github.com/patrick-electrick")
+	)
 	(junction
 		(at 86.36 130.81)
@@
 	)
 	(label "POT2"
-		(at 204.47 96.52 180)
+		(at 204.47 101.6 180)
 		(effects
 			(font
@@
 	)
 	(label "POT4"
-		(at 204.47 101.6 180)
+		(at 204.47 96.52 180)
 		(effects
 			(font
@@
 	)
 	(label "POT1"
-		(at 204.47 93.98 180)
+		(at 204.47 104.14 180)
 		(effects
 			(font
@@
 	)
 	(label "POT5"
-		(at 204.47 104.14 180)
-		(effects
-			(font
+		(at 204.47 93.98 180)
+		(effects
+			(font
