File: hardware/KiCad/schematics/output_buffer.kicad_sch (KiCad schematic)
At the start: 12 parts, among them U2 MCP6022

Commit message: Added identification properties for KiCad schematic drawing sheets.
Other:
- company: (none) -> github.com/patrick-electrick
- title: (none) -> MIMEOFREQ
Changed lines of the file:
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@@
 	(generator_version "10.0")
 	(paper "A4")
+	(title_block
+		(title "MIMEOFREQ")
+		(date "2026-10-21")
+		(rev "1")
+		(company "github.com/patrick-electrick")
+	)
 	(junction
 		(at 120.65 111.76)
